File: HW/GH_Terra_pre.sch (EAGLE design)
At the start: 23 parts, among them IC1 STM32F030C6T

Commit message: Почти полная версия.
Parts:
- removed G1: VST3, battery:VST3
- removed IC1: STM32F030C6T, micro-stm:STM32F030C6T
- removed LCD: (no value), con-lstb:MA08-2
- removed PIN1, PIN2: (no value), wirepad:2,15/1,0
- added C10: CC0603JRX7R9BB104, rcl:C-EUC0603
- added C11: CC0603KRX5R7BB105, rcl:C-EUC0603
- added C5, C6, C7, C8, C9: CC0603GRNPO9BN220, rcl:C-EUC0603
- added D1, D2: ESDA14V2L, diode:BAS40-06
- added L1: BLM18AG102SN1D, rcl:L-US
- added LCD1: CHT2623, lcd_glass:CHT2623
- added PAD1, PAD2: (no value), wirepad:2,54/1,0
- added Q1, Q4: IRLML5203TRPBF, semiconductor:PFET-SOT23
- added Q2, Q5: IRLML2030TRPBF, semiconductor:NFET-SOT23
- added Q3: 16MHz, crystal:CRYTALHC49S
- added Q6, Q7: BC817-40.215, semicon-smd-ipc:NPN-TRANSISTOR_SOT23
- added R10, R11, R12, R13: RC0603FR-0727KL, rcl:R-EU_R0603
- added R14, R18: RC0603JR-079R1L, rcl:R-EU_R0603
- added R15: CRCW06031K00JNEA, rcl:R-EU_R0603
- added R16, R17, R19: RC0603FR-07100KL, rcl:R-EU_R0603
- added R20, R21, R22, R23, R24, R25, R26: CR0603-FX-1002ELF, rcl:R-EU_R0603
- added SV1: (no value), con-lstb:MA04-1
- added SV2: (no value), con-lstb:MA03-1
- added U$6: MA02-1, con-lstb:MA02-1
- added U1: STM8L152C6T6, st-microelectronics:STM8L152C6
- C1, C2: value (none) -> CC0603JRX7R9BB104
- C3: value (none) -> SH063M0010B2F-0511; device rcl:CPOL-EUD/7343-31R -> rcl:CPOL-EUSANYO_C6
- C4: value (none) -> CC0603GRNPO9BN220
- R1: value (none) -> RC0603JR-0710RL
- R2: value (none) -> B57621C0103J062; device rcl:R-EU_R0603 -> rcl:R-EU_R1206
- R3: value (none) -> CR0603-FX-1002ELF
- R4, R5: value (none) -> RC0603FR-0727KL
- R6, R7, R8, R9: value (none) -> RC0603FR-07100KL
- U$1: value KX-327LT -> MA02-1; device crystal:KX-327LT -> con-lstb:MA02-1
- U$2, U$3, U$4, U$5: value SWT-32 -> (none); device ohranyator:SWT-32 -> rubber_key:RK_4X3
Connections:
- removed net N$5: IC1MCU.PB15, LCD.16
- new net MCC: R15.1, U1.PD7
- new net N$22: LCD1.SEG11, U1.PB1/TIM3_CH1/LCD_SEG11/ADC1_IN17/COMP1_INP
- new net N$27: D2.K1, D2.K2, PAD2.P, R11.1, R13.1, U1.PD4/TIM1_CH2
- new net N$28: R10.2, R12.2, U1.PD5/TIM1_CH3
- new net N$29: LCD1.SEG16, U1.PB6/LCD_SEG16/ADC1_IN12/COMP1_INP
- new net N$30: C4.1, R6.1, U$2.P, U1.PC0
- new net N$31: C5.1, R7.1, U$3.P, U1.PC1
- new net N$32: C7.1, R8.1, U$4.P, U1.PC5
- new net N$33: C8.1, R9.1, U$5.P, U1.PC6
- new net N$34: LCD1.SEG17, U1.PB7/LCD_SEG17/ADC1_IN11/COMP1_INP
- new net N$35: Q6.B, Q7.C, R15.2
- new net POWER_TEMP: R3.1, U1.PF0/ADC1_IN24/DAC_OUT
- new net RESET: R17.2, SV1.4, U1.NRST/PA1
- new net SWIM: SV1.2, U1.PA0/SWIM/BEEP/IR_TIM
- new net TEMP_ADC: R2.1, R3.2, U1.PD6
- new net USART_RX: R16.1, SV2.2, U1.PC2/USART1_RX
- new net USART_TX: SV2.1, U1.PC3/USART1_TX
- new net VALVE_CLOSE: Q4.G, Q5.G, R5.1, U1.PE7
- new net VALVE_OPEN: Q1.G, Q2.G, R4.2, U1.PE6
- new net VLCD: C11.1, U1.VLCD
- new net VREF: R10.1, R11.2, R19.2, R20.1, R24.1, U1.PC7/ADC1_IN3
- new net VREF+: R20.2, R21.1, R22.1, R23.2, U1.VREF+
- new net VREF-: R24.2, R25.2, R26.1, U1.VSS1/VSSA/VREF-
- new net VREF1: D1.K1, D1.K2, PAD1.P, R12.1, R13.2, R21.2, R25.1, U1.PC4/ADC1_IN4
- new net VREF2: C2.1, L1.1, R19.1, R23.1, U1.VDDA
- new net XTAL_IN: C6.1, Q3.2, U1.PA2/OSC_IN
- new net XTAL_OUT: C9.1, Q3.1, U1.PA3/OSC_OUT
- net GND: now also C11.2, C4.2, C5.2, C6.2, C7.2, C8.2, C9.2, D1.AA, D2.AA, Q7.E, R14.2, R18.2, R2.2, R26.2, SV1.3, SV2.3, U$2.S, U$3.S, U$4.S, U$5.S, U$6.2, U1.VSS2; no longer G1.-, IC1MCU.VSSA, U$2.1, U$3.1, U$4.1, U$5.1
- net N$1: now also Q1.S, Q4.S, R1.2; no longer C4.1, IC1MCU.PA7, R3.2, R4.1
- net N$10: now also LCD1.COM4, U1.PD1/LCD_COM3; no longer IC1MCU.NRST, R1.1
- net N$11: now also LCD1.SEG0, U1.PA7/LCD_SEG0; no longer IC1MCU.PB14, LCD.14
- net N$12: now also LCD1.SEG1, U1.PE0/LCD_SEG1; no longer IC1MCU.PB13, LCD.12
- net N$13: now also LCD1.SEG2, U1.PE1/TIM1_CH2N/LCD_SEG2; no longer IC1MCU.PB12, LCD.10
- net N$14: now also LCD1.SEG3, U1.PE2/TIM1_CH3N/LCD_SEG3; no longer IC1MCU.PB11, LCD.8
- net N$15: now also LCD1.SEG4, U1.PE3/LCD_SEG4; no longer IC1MCU.PB10, LCD.6
- net N$16: now also LCD1.SEG5, U1.PE4/LCD_SEG5; no longer IC1MCU.PB9, LCD.4
- net N$17: now also LCD1.SEG6, U1.PE5/LCD_SEG6/ADC1_IN23/COMP2_INP/COMP1_INP; no longer IC1MCU.PB8, LCD.2
- net N$18: now also LCD1.SEG7, U1.PD0/TIM3_CH2/LCD_SEG7/ADC1_IN22/COMP2_INP/COMP1_INP; no longer IC1MCU.PB6, LCD.1
- net N$19: now also LCD1.SEG8, U1.PD2/TIM1_CH1/LCD_SEG8/ADC1_IN20/COMP1_INP; no longer IC1MCU.PB5, LCD.3
- net N$2: now also C10.1, Q1.D, Q2.D, U$1.2; no longer C3.+, G1.+, IC1MCU.VDDA
- net N$20: now also LCD1.SEG9, U1.PD3/TIM1_ETR/LCD_SEG9/ADC1_IN19/COMP1_INP; no longer IC1MCU.PB4, LCD.5
- net N$21: now also LCD1.SEG10, U1.PB0/TIM2_CH1/LCD_SEG10/ADC1_IN18/COMP1_INP; no longer IC1MCU.PB3, LCD.7
- net N$23: now also LCD1.SEG12, U1.PB2/TIM2_CH2/LCD_SEG12/ADC1_IN16/COMP1_INP; no longer IC1MCU.PB2, R6.2, U$2.3
- net N$24: now also LCD1.SEG13, U1.PB3/TIM2_ETR/LCD_SEG13/ADC1_IN15/COMP1_INP; no longer IC1MCU.PB1, R7.2, U$3.3
- net N$25: now also LCD1.SEG14, U1.PB4/LCD_SEG14/ADC1_IN14/COMP1_INP; no longer IC1MCU.PB0, R8.2, U$4.3
- net N$26: now also LCD1.SEG15, U1.PB5/LCD_SEG15/AD1_IN13/COMP1_INP; no longer IC1MCU.PA15, R9.2, U$5.3
- net N$3: now also C10.2, Q4.D, Q5.D; no longer C1.1, IC1MCU.OSC_IN
- net N$4: now also Q2.S, Q5.S, Q6.C, R4.1, R5.2; no longer C2.1, IC1MCU.OSC_OUT, U$1.2
- net N$6: now also Q6.E, Q7.B, R14.1, R18.1; no longer IC1MCU.PA3, R3.1, R5.1
- net N$7: now also LCD1.COM1, U1.PA4/LCD_COM0/; no longer C4.2, IC1MCU.PA1, PIN1.P, R5.2
- net N$8: now also LCD1.COM2, U1.PA5/LCD_COM1; no longer IC1MCU.PA8, PIN2.P, R4.2
- net N$9: now also LCD1.COM3, U1.PA6/LCD_COM2; no longer IC1MCU.BOOT0, R2.1
- net VCC: now also C1.1, C3.+, L1.2, R1.1, R16.2, R17.1, R22.2, R6.2, R7.2, R8.2, R9.2, SV1.1, U$6.1, U1.VDD, U1.VDD2; no longer R1.2, R2.2, R6.1, R7.1, R8.1, R9.1
Other:
- note added: "150mA"
- note added: "Battary"
- note added: "DOWN"
- note added: "In=0.66/R2"
- note added: "SENSOR"
- note added: "SET"
- note added: "SWIM"
- note added: "UP"
- note added: "USART"
- note added: "VALVE"
- note added: "VALVE OPEN/CLOSE"
- note added: "calcResult_for_termistor.csv"
- note added: "t°"
- moved on the sheet: C1, C2, C3, C4, R1, R2, R3, R4, R5, R6, R7, R8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

Commit message: REV1
Parts:
- removed C10: CC0603JRX7R9BB104, rcl:C-EUC0603
- removed C6, C8, C9: CC0603GRNPO9BN220, rcl:C-EUC0603
- removed L1: BLM18AG102SN1D, rcl:L-US
- removed PAD1, PAD2: (no value), wirepad:2,54/1,0
- removed Q3: 16MHz, crystal:CRYTALHC49S
- removed Q6, Q7: BC817-40.215, semicon-smd-ipc:NPN-TRANSISTOR_SOT23
- removed R1: RC0603JR-0710RL, rcl:R-EU_R0603
- removed R14, R18: RC0603JR-079R1L, rcl:R-EU_R0603
- removed R15: CRCW06031K00JNEA, rcl:R-EU_R0603
- removed R16, R19, R9: RC0603FR-07100KL, rcl:R-EU_R0603
- removed R20, R21, R22, R23, R24, R25, R26: CR0603-FX-1002ELF, rcl:R-EU_R0603
- removed SV2: (no value), con-lstb:MA03-1
- U$5: value (none) -> MA02-1; device rubber_key:RK_4X3 -> con-lstb:MA02-1
Connections:
- removed net N$1: Q1.S, Q4.S, R1.2
- removed net N$33: C8.1, R9.1, U$5.P, U1.PC6
- removed net N$35: Q6.B, Q7.C, R15.2
- removed net N$4: Q2.S, Q5.S, Q6.C, R4.1, R5.2
- removed net N$6: Q6.E, Q7.B, R14.1, R18.1
- removed net USART_RX: R16.1, SV2.2, U1.PC2/USART1_RX
- removed net USART_TX: SV2.1, U1.PC3/USART1_TX
- removed net VREF-: R24.2, R25.2, R26.1, U1.VSS1/VSSA/VREF-
- removed net VREF2: C2.1, L1.1, R19.1, R23.1, U1.VDDA
- removed net XTAL_IN: C6.1, Q3.2, U1.PA2/OSC_IN
- removed net XTAL_OUT: C9.1, Q3.1, U1.PA3/OSC_OUT
- net GND: now also Q2.S, Q5.S, R4.1, R5.2, U1.VSS1/VSSA/VREF-; no longer C6.2, C8.2, C9.2, Q7.E, R14.2, R18.2, R26.2, SV2.3, U$5.S
- net MCC: no longer R15.1
- net N$2: no longer C10.1
- net N$27: now also U$5.1; no longer PAD2.P
- net N$3: no longer C10.2
- net VCC: now also C2.1, Q1.S, Q4.S, U1.VDDA; no longer L1.2, R1.1, R16.2, R22.2, R9.2
- net VREF: no longer R19.2, R20.1, R24.1
- net VREF+: no longer R20.2, R21.1, R22.1, R23.2
- net VREF1: now also U$5.2; no longer PAD1.P, R21.2, R25.1
Other:
- note removed: "150mA"
- note removed: "In=0.66/R2"
- note removed: "USART"
- note removed: "VALVE OPEN/CLOSE"

Commit message: Закостылили мерцание показаний датчика влажности. Гореть мне в Аду за это....
Parts:
- added C6: CC0603JRX7R9BB104, rcl:C-EUC0603
- added R1: RC0603FR-07100KL, rcl:R-EU_R0603
- added U7: MA02-1, con-lstb:MA02-1
- Q1, Q4: value IRLML5203TRPBF -> IRLML6402
- Q2, Q5: value IRLML2030TRPBF -> IRLML6244
Connections:
- removed net MCC: U1.PD7
- removed net VREF+: U1.VREF+
- new net CHECK_POS: R1.1, U1.PA3/OSC_OUT
- new net STATE: C6.1, R1.2, U1.PD7, U7.1
- net GND: now also C6.2, U7.2
- net VCC: now also U1.VREF+
Other:
- note added: "SENSOR_OF_POSITION"
Changed lines of the file:
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@@
 <layer number="94" name="Symbols" color="4" fill="1" visible="yes" active="yes"/>
 <layer number="95" name="Names" color="7" fill="1" visible="yes" active="yes"/>
-<layer number="96" name="Values" color="7" fill="1" visible="no" active="yes"/>
+<layer number="96" name="Values" color="7" fill="1" visible="yes" active="yes"/>
 <layer number="97" name="Info" color="7" fill="1" visible="yes" active="yes"/>
 <layer number="98" name="Guide" color="6" fill="1" visible="yes" active="yes"/>
@@
 <part name="GND2" library="supply1" deviceset="GND" device=""/>
 <part name="GND3" library="supply1" deviceset="GND" device=""/>
-<part name="Q1" library="semiconductor" deviceset="PFET-" device="SOT23" value="IRLML5203TRPBF"/>
-<part name="Q4" library="semiconductor" deviceset="PFET-" device="SOT23" value="IRLML5203TRPBF"/>
-<part name="Q5" library="semiconductor" deviceset="NFET-" device="SOT23" value="IRLML2030TRPBF"/>
-<part name="Q2" library="semiconductor" deviceset="NFET-" device="SOT23" value="IRLML2030TRPBF"/>
+<part name="Q1" library="semiconductor" deviceset="PFET-" device="SOT23" value="IRLML6402"/>
+<part name="Q4" library="semiconductor" deviceset="PFET-" device="SOT23" value="IRLML6402"/>
+<part name="Q5" library="semiconductor" deviceset="NFET-" device="SOT23" value="IRLML6244"/>
+<part name="Q2" library="semiconductor" deviceset="NFET-" device="SOT23" value="IRLML6244"/>
 <part name="R4" library="rcl" deviceset="R-EU_" device="R0603" value="RC0603FR-0727KL"/>
 <part name="R5" library="rcl" deviceset="R-EU_" device="R0603" value="RC0603FR-0727KL"/>
@@
 <part name="GND4" library="supply1" deviceset="GND" device=""/>
 <part name="U$5" library="con-lstb" deviceset="MA02-1" device=""/>
+<part name="R1" library="rcl" deviceset="R-EU_" device="R0603" value="RC0603FR-07100KL"/>
+<part name="C6" library="rcl" deviceset="C-EU" device="C0603" value="CC0603JRX7R9BB104"/>
+<part name="GND5" library="supply1" deviceset="GND" device=""/>
+<part name="U7" library="con-lstb" deviceset="MA02-1" device=""/>
+<part name="GND10" library="supply1" deviceset="GND" device=""/>
 </parts>
 <sheets>
@@
 <text x="248.92" y="12.7" size="1.6764" layer="91" rot="R90">DOWN</text>
 <frame x1="-198.12" y1="-175.26" x2="302.26" y2="88.9" columns="8" rows="5" layer="97"/>
+<text x="251.46" y="-134.62" size="1.778" layer="91">SENSOR_OF_POSITION</text>
 </plain>
 <instances>
@@
 <instance part="GND4" gate="1" x="2.54" y="-139.7"/>
 <instance part="U$5" gate="G$1" x="144.78" y="-139.7" rot="R90"/>
+<instance part="R1" gate="G$1" x="231.14" y="-124.46" rot="R270"/>
+<instance part="C6" gate="G$1" x="231.14" y="-137.16" smashed="yes">
+<attribute name="NAME" x="232.664" y="-136.779" size="1.778" layer="95"/>
+<attribute name="VALUE" x="234.061" y="-138.684" size="1.778" layer="96" rot="R270"/>
+</instance>
+<instance part="GND5" gate="1" x="231.14" y="-147.32" smashed="yes">
+<attribute name="VALUE" x="228.6" y="-149.86" size="1.778" layer="96"/>
+</instance>
+<instance part="U7" gate="G$1" x="248.92" y="-134.62" rot="R180"/>
+<instance part="GND10" gate="1" x="241.3" y="-147.32" smashed="yes">
+<attribute name="VALUE" x="238.76" y="-149.86" size="1.778" layer="96"/>
+</instance>
 </instances>
 <busses>
@@
 <pinref part="GND4" gate="1" pin="GND"/>
 </segment>
+<segment>
+<pinref part="C6" gate="G$1" pin="2"/>
+<pinref part="GND5" gate="1" pin="GND"/>
+<wire x1="231.14" y1="-142.24" x2="231.14" y2="-144.78" width="0.1524" layer="91"/>
+</segment>
+<segment>
+<pinref part="U7" gate="G$1" pin="2"/>
+<pinref part="GND10" gate="1" pin="GND"/>
+<wire x1="241.3" y1="-134.62" x2="241.3" y2="-144.78" width="0.1524" layer="91"/>
+</segment>
 </net>
 <net name="VCC" class="0">
@@
 <wire x1="195.58" y1="25.4" x2="195.58" y2="27.94" width="0.1524" layer="91"/>
 <label x="195.58" y="27.94" size="1.016" layer="95" rot="R90" xref="yes"/>
-</segment>
-<segment>
-<pinref part="U1" gate="G$1" pin="VDD"/>
-<wire x1="91.44" y1="45.72" x2="101.6" y2="45.72" width="0.1524" layer="91"/>
-<wire x1="101.6" y1="45.72" x2="101.6" y2="43.18" width="0.1524" layer="91"/>
-<pinref part="U1" gate="G$1" pin="VDD2"/>
-<wire x1="101.6" y1="43.18" x2="101.6" y2="40.64" width="0.1524" layer="91"/>
-<wire x1="101.6" y1="40.64" x2="91.44" y2="40.64" width="0.1524" layer="91"/>
-<wire x1="101.6" y1="43.18" x2="106.68" y2="43.18" width="0.1524" layer="91"/>
-<pinref part="C1" gate="G$1" pin="1"/>
-<wire x1="106.68" y1="43.18" x2="106.68" y2="40.64" width="0.1524" layer="91"/>
-<wire x1="106.68" y1="43.18" x2="109.22" y2="43.18" width="0.1524" layer="91"/>
-<junction x="106.68" y="43.18"/>
-<junction x="101.6" y="43.18"/>
-<label x="109.22" y="43.18" size="1.016" layer="95" xref="yes"/>
 </segment>
 <segment>
@@
 <wire x1="-88.9" y1="-76.2" x2="-96.52" y2="-76.2" width="0.1524" layer="91"/>
 <label x="-96.52" y="-76.2" size="1.016" layer="95" rot="R180" xref="yes"/>
+</segment>
+<segment>
+<pinref part="U1" gate="G$1" pin="VREF+"/>
+<wire x1="91.44" y1="35.56" x2="101.6" y2="35.56" width="0.1524" layer="91"/>
+<pinref part="U1" gate="G$1" pin="VDD"/>
+<wire x1="91.44" y1="45.72" x2="101.6" y2="45.72" width="0.1524" layer="91"/>
+<wire x1="101.6" y1="45.72" x2="101.6" y2="43.18" width="0.1524" layer="91"/>
+<pinref part="U1" gate="G$1" pin="VDD2"/>
+<wire x1="101.6" y1="43.18" x2="101.6" y2="40.64" width="0.1524" layer="91"/>
+<wire x1="101.6" y1="40.64" x2="91.44" y2="40.64" width="0.1524" layer="91"/>
+<wire x1="101.6" y1="43.18" x2="106.68" y2="43.18" width="0.1524" layer="91"/>
+<pinref part="C1" gate="G$1" pin="1"/>
+<wire x1="106.68" y1="43.18" x2="106.68" y2="40.64" width="0.1524" layer="91"/>
+<wire x1="106.68" y1="43.18" x2="109.22" y2="43.18" width="0.1524" layer="91"/>
+<junction x="106.68" y="43.18"/>
+<junction x="101.6" y="43.18"/>
+<label x="109.22" y="43.18" size="1.016" layer="95" xref="yes"/>
+<wire x1="101.6" y1="35.56" x2="101.6" y2="40.64" width="0.1524" layer="91"/>
+<junction x="101.6" y="40.64"/>
 </segment>
 </net>
@@
 </segment>
 </net>
-<net name="VREF+" class="0">
-<segment>
-<pinref part="U1" gate="G$1" pin="VREF+"/>
-<wire x1="91.44" y1="35.56" x2="93.98" y2="35.56" width="0.1524" layer="91"/>
-<label x="93.98" y="35.56" size="1.016" layer="95" xref="yes"/>
-</segment>
-</net>
 <net name="N$2" class="0">
 <segment>
@@
 </segment>
 </net>
-<net name="MCC" class="0">
+<net name="STATE" class="0">
 <segment>
 <pinref part="U1" gate="G$1" pin="PD7"/>
 <wire x1="91.44" y1="20.32" x2="121.92" y2="20.32" width="0.1524" layer="91"/>
 <label x="121.92" y="20.32" size="1.016" layer="95" xref="yes"/>
+</segment>
+<segment>
+<pinref part="R1" gate="G$1" pin="2"/>
+<pinref part="C6" gate="G$1" pin="1"/>
+<wire x1="231.14" y1="-129.54" x2="231.14" y2="-132.08" width="0.1524" layer="91"/>
+<wire x1="231.14" y1="-132.08" x2="231.14" y2="-134.62" width="0.1524" layer="91"/>
+<wire x1="231.14" y1="-132.08" x2="223.52" y2="-132.08" width="0.1524" layer="91"/>
+<wire x1="231.14" y1="-132.08" x2="241.3" y2="-132.08" width="0.1524" layer="91"/>
+<junction x="231.14" y="-132.08"/>
+<label x="223.52" y="-132.08" size="1.778" layer="95" rot="R180" xref="yes"/>
+<pinref part="U7" gate="G$1" pin="1"/>
 </segment>
 </net>
@@
 <pinref part="R17" gate="G$1" pin="2"/>
 <wire x1="-86.36" y1="-50.8" x2="-88.9" y2="-50.8" width="0.1524" layer="91"/>
-<wire x1="-86.36" y1="-50.8" x2="-86.36" y2="-53.34" width="0.1524" layer="91"/>
+<wire x1="-86.36" y1="-50.8" x2="-86.36" y2="-55.88" width="0.1524" layer="91"/>
 <junction x="-86.36" y="-50.8"/>
-<label x="-86.36" y="-53.34" size="1.016" layer="95" rot="R270" xref="yes"/>
+<label x="-86.36" y="-55.88" size="1.016" layer="95" rot="R270" xref="yes"/>
 </segment>
 </net>
@@
 </segment>
 </net>
+<net name="CHECK_POS" class="0">
+<segment>
+<pinref part="U1" gate="G$1" pin="PA3/OSC_OUT"/>
+<wire x1="91.44" y1="55.88" x2="96.52" y2="55.88" width="0.1524" layer="91"/>
+<label x="96.52" y="55.88" size="1.778" layer="95" xref="yes"/>
+</segment>
+<segment>
+<pinref part="R1" gate="G$1" pin="1"/>
+<wire x1="231.14" y1="-119.38" x2="231.14" y2="-114.3" width="0.1524" layer="91"/>
+<label x="231.14" y="-114.3" size="1.778" layer="95" rot="R90" xref="yes"/>
+</segment>
+</net>
